File: UVLEDController/UVLEDController/UVLEDController.kicad_sch (KiCad schematic)
At the start: 15 parts, among them J1 Screw_Terminal_01x02, J2 Screw_Terminal_01x02, J3 Conn_01x04_Male, Q1 Q_NMOS_GDS

Commit message: Updates for physical dimensions based on Fuseion360 test fits.
Parts:
- H1, H2, H3, H4, H5, H6: footprint MountingHole:MountingHole_3.2mm_M3_DIN965 -> MountingHole:MountingHole_3mm
Changed lines of the file:
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@@
       (effects (font (size 1.27 1.27)) (justify left))
     )
-    (property "Footprint" "MountingHole:MountingHole_3.2mm_M3_DIN965" (id 2) (at 59.69 106.68 0)
+    (property "Footprint" "MountingHole:MountingHole_3mm" (id 2) (at 59.69 106.68 0)
       (effects (font (size 1.27 1.27)) hide)
     )
@@
       (effects (font (size 1.27 1.27)) (justify left))
     )
-    (property "Footprint" "MountingHole:MountingHole_3.2mm_M3_DIN965" (id 2) (at 59.69 96.52 0)
+    (property "Footprint" "MountingHole:MountingHole_3mm" (id 2) (at 59.69 96.52 0)
       (effects (font (size 1.27 1.27)) hide)
     )
@@
       (effects (font (size 1.27 1.27)) (justify left))
     )
-    (property "Footprint" "MountingHole:MountingHole_3.2mm_M3_DIN965" (id 2) (at 59.69 111.76 0)
+    (property "Footprint" "MountingHole:MountingHole_3mm" (id 2) (at 59.69 111.76 0)
       (effects (font (size 1.27 1.27)) hide)
     )
@@
       (effects (font (size 1.27 1.27)) (justify left))
     )
-    (property "Footprint" "MountingHole:MountingHole_3.2mm_M3_DIN965" (id 2) (at 59.69 101.6 0)
+    (property "Footprint" "MountingHole:MountingHole_3mm" (id 2) (at 59.69 101.6 0)
       (effects (font (size 1.27 1.27)) hide)
     )
@@
       (effects (font (size 1.27 1.27)) (justify left))
     )
-    (property "Footprint" "MountingHole:MountingHole_3.2mm_M3_DIN965" (id 2) (at 59.69 116.84 0)
+    (property "Footprint" "MountingHole:MountingHole_3mm" (id 2) (at 59.69 116.84 0)
       (effects (font (size 1.27 1.27)) hide)
     )
@@
       (effects (font (size 1.27 1.27)) (justify left))
     )
-    (property "Footprint" "MountingHole:MountingHole_3.2mm_M3_DIN965" (id 2) (at 59.69 91.44 0)
+    (property "Footprint" "MountingHole:MountingHole_3mm" (id 2) (at 59.69 91.44 0)
       (effects (font (size 1.27 1.27)) hide)
     )
@@
     )
     (path "/f2ac6cc0-0296-45c7-b704-04cf6e9cafbf"
-      (reference "H1") (unit 1) (value "MountingHole") (footprint "MountingHole:MountingHole_3.2mm_M3_DIN965")
+      (reference "H1") (unit 1) (value "MountingHole") (footprint "MountingHole:MountingHole_3mm")
     )
     (path "/22a71b48-1255-4c52-9487-a7d01be309d7"
-      (reference "H2") (unit 1) (value "MountingHole") (footprint "MountingHole:MountingHole_3.2mm_M3_DIN965")
+      (reference "H2") (unit 1) (value "MountingHole") (footprint "MountingHole:MountingHole_3mm")
     )
     (path "/b81eaa30-7386-49a4-a4b1-a10a128eb59e"
-      (reference "H3") (unit 1) (value "MountingHole") (footprint "MountingHole:MountingHole_3.2mm_M3_DIN965")
+      (reference "H3") (unit 1) (value "MountingHole") (footprint "MountingHole:MountingHole_3mm")
     )
     (path "/0c2fe7c3-99b0-4a57-9104-9889649d577f"
-      (reference "H4") (unit 1) (value "MountingHole") (footprint "MountingHole:MountingHole_3.2mm_M3_DIN965")
+      (reference "H4") (unit 1) (value "MountingHole") (footprint "MountingHole:MountingHole_3mm")
     )
     (path "/58a46c49-40db-462e-b695-557061bc8968"
-      (reference "H5") (unit 1) (value "MountingHole") (footprint "MountingHole:MountingHole_3.2mm_M3_DIN965")
+      (reference "H5") (unit 1) (value "MountingHole") (footprint "MountingHole:MountingHole_3mm")
     )
     (path "/cabe01f1-3803-4bbd-a53f-5d2860a51920"
-      (reference "H6") (unit 1) (value "MountingHole") (footprint "MountingHole:MountingHole_3.2mm_M3_DIN965")
+      (reference "H6") (unit 1) (value "MountingHole") (footprint "MountingHole:MountingHole_3mm")
     )
     (path "/b199a8ce-ac04-4537-a164-631a8a6e80cd"

Commit message: Moved the buttons to below the screen.
Parts:
- removed H5, H6: MountingHole, MountingHole:MountingHole_3mm, symbol Mechanical:MountingHole
Changed lines of the file:
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@@
     (pin "1")
-  )
-  (symbol (lib_id "Mechanical:MountingHole") (at 59.69 111.76 0) (unit 1)
-    (in_bom yes) (on_board yes) (fields_autoplaced)
-    (property "Reference" "H5" (id 0) (at 62.23 110.9253 0)
-      (effects (font (size 1.27 1.27)) (justify left))
-    )
-    (property "Value" "MountingHole" (id 1) (at 62.23 113.4622 0)
-      (effects (font (size 1.27 1.27)) (justify left))
-    )
-    (property "Footprint" "MountingHole:MountingHole_3mm" (id 2) (at 59.69 111.76 0)
-      (effects (font (size 1.27 1.27)) hide)
-    )
-    (property "Datasheet" "~" (id 3) (at 59.69 111.76 0)
-      (effects (font (size 1.27 1.27)) hide)
-    )
   )
   (symbol (lib_id "Device:Q_NMOS_GDS") (at 34.29 80.01 0) (mirror y) (unit 1)
@@
     (pin "2")
   )
-  (symbol (lib_id "Mechanical:MountingHole") (at 59.69 116.84 0) (unit 1)
-    (in_bom yes) (on_board yes) (fields_autoplaced)
-    (property "Reference" "H6" (id 0) (at 62.23 116.0053 0)
-      (effects (font (size 1.27 1.27)) (justify left))
-    )
-    (property "Value" "MountingHole" (id 1) (at 62.23 118.5422 0)
-      (effects (font (size 1.27 1.27)) (justify left))
-    )
-    (property "Footprint" "MountingHole:MountingHole_3mm" (id 2) (at 59.69 116.84 0)
-      (effects (font (size 1.27 1.27)) hide)
-    )
-    (property "Datasheet" "~" (id 3) (at 59.69 116.84 0)
-      (effects (font (size 1.27 1.27)) hide)
-    )
-  )
   (symbol (lib_id "power:GND") (at 86.36 20.32 0) (unit 1)
     (in_bom yes) (on_board yes) (fields_autoplaced)
@@
       (reference "H4") (unit 1) (value "MountingHole") (footprint "MountingHole:MountingHole_3mm")
     )
-    (path "/58a46c49-40db-462e-b695-557061bc8968"
-      (reference "H5") (unit 1) (value "MountingHole") (footprint "MountingHole:MountingHole_3mm")
-    )
-    (path "/cabe01f1-3803-4bbd-a53f-5d2860a51920"
-      (reference "H6") (unit 1) (value "MountingHole") (footprint "MountingHole:MountingHole_3mm")
-    )
     (path "/b199a8ce-ac04-4537-a164-631a8a6e80cd"

Commit message: Moved the screw terminals to a better location. Tweaked position of i2c header.
Parts:
- renumbered J1 to J1-LED1, J2 to J2-PWR1
Changed lines of the file:
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@@
   (symbol (lib_id "Connector:Screw_Terminal_01x02") (at 60.96 13.97 90) (unit 1)
     (in_bom yes) (on_board yes) (fields_autoplaced)
-    (property "Reference" "J2" (id 0) (at 65.532 13.1353 90)
+    (property "Reference" "J2-PWR1" (id 0) (at 65.532 13.1353 90)
       (effects (font (size 1.27 1.27)) (justify right))
     )
@@
   (symbol (lib_id "Connector:Screw_Terminal_01x02") (at 20.32 72.39 0) (mirror y) (unit 1)
     (in_bom yes) (on_board yes) (fields_autoplaced)
-    (property "Reference" "J1" (id 0) (at 20.32 67.4202 0))
+    (property "Reference" "J1-LED1" (id 0) (at 20.32 67.4202 0))
     (property "Value" "Screw_Terminal_01x02" (id 1) (at 20.32 69.9571 0))
     (property "Footprint" "TerminalBlock_Phoenix:TerminalBlock_Phoenix_PT-1,5-2-5.0-H_1x02_P5.00mm_Horizontal" (id 2) (at 20.32 72.39 0)
@@
     )
     (path "/b199a8ce-ac04-4537-a164-631a8a6e80cd"
-      (reference "J1") (unit 1) (value "Screw_Terminal_01x02") (footprint "TerminalBlock_Phoenix:TerminalBlock_Phoenix_PT-1,5-2-5.0-H_1x02_P5.00mm_Horizontal")
+      (reference "J1-LED1") (unit 1) (value "Screw_Terminal_01x02") (footprint "TerminalBlock_Phoenix:TerminalBlock_Phoenix_PT-1,5-2-5.0-H_1x02_P5.00mm_Horizontal")
     )
     (path "/43944736-18ad-462d-858d-dfa0358b53b3"
-      (reference "J2") (unit 1) (value "Screw_Terminal_01x02") (footprint "TerminalBlock_Phoenix:TerminalBlock_Phoenix_PT-1,5-2-5.0-H_1x02_P5.00mm_Horizontal")
+      (reference "J2-PWR1") (unit 1) (value "Screw_Terminal_01x02") (footprint "TerminalBlock_Phoenix:TerminalBlock_Phoenix_PT-1,5-2-5.0-H_1x02_P5.00mm_Horizontal")
     )
     (path "/24d1c1f3-5055-473a-85cc-45ac6541ea90"
